File: Schematics/FerrantiPC33.kicad_sch (KiCad schematic)
At the start: 63 parts, among them J1 ULA 5RA022E-2, J2 Bus_ISA_8bit, J3 ULA 5RA023EE-2, J5914 AM2966, U1 74LS14, U10 8288, U11 8086_Max_Mode, U12 74LS00, U13 8255, U14 8237, U15 74LS74, U16 74LS670, U17 74LS00, U18 PAL16L8 - BUS CONV?, U19 PAL16L8, U2 74LS08, U20 74LS74, U21 74LS32, U22 27128, U24 74LS20, U26 74LS244, U27 74LS244, U28 74LS245, U29 74LS244, U3 8250, U30 74LS245, U32 74LS280, U4 74LS193, U5 74LS04, U5204 74LS245, U5211 74LS373, U5311 74LS373, U5403 74LS125, U5405 74LS244, U5411 74LS373, U5504 74LS04, U5611 74LS245, U5612 74LS245, U5715 74LS245, U5819 74LS32, U5820 EP8202_DELAY_LINE, U5821 74LS00, U5917 74LS373, U5919 74LS32, U6 8253, U6015 74LS245, U6018 74LS280, U6020 74LS32, U6119 41256 DRAM, U6218 41256 DRAM, U6219 41256 DRAM, U7 8087, U8 27128, U9 8284, Y1 Crystal

Commit message: Adding a lot more of the things I've collected about this board.
Other:
- note removed: "It's LOW that's not right?"
Changed lines of the file:
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@@
 	(wire
 		(pts
-			(xy 207.01 354.33) (xy 212.09 354.33)
-		)
-		(stroke
-			(width 0)
-			(type default)
-		)
-	)
-	(wire
-		(pts
 			(xy 68.58 55.88) (xy 60.96 55.88)
 		)
@@
 	(wire
 		(pts
-			(xy 149.86 354.33) (xy 152.4 354.33)
+			(xy 34.29 344.17) (xy 139.7 344.17)
 		)
 		(stroke
@@
 	(wire
 		(pts
+			(xy 139.7 359.41) (xy 152.4 359.41)
+		)
+		(stroke
+			(width 0)
+			(type default)
+		)
+	)
+	(wire
+		(pts
 			(xy 565.15 124.46) (xy 551.18 124.46)
 		)
@@
 		)
 	)
-	(polyline
-		(pts
-			(xy 148.59 345.44) (xy 148.59 350.52)
-		)
-		(stroke
-			(width 0)
-			(type default)
-		)
-	)
 	(wire
 		(pts
@@
 	(wire
 		(pts
+			(xy 35.56 369.57) (xy 152.4 369.57)
+		)
+		(stroke
+			(width 0)
+			(type default)
+		)
+	)
+	(wire
+		(pts
 			(xy 214.63 476.25) (xy 217.17 476.25)
 		)
@@
 	(wire
 		(pts
+			(xy 139.7 344.17) (xy 139.7 354.33)
+		)
+		(stroke
+			(width 0)
+			(type default)
+		)
+	)
+	(wire
+		(pts
 			(xy 161.29 139.7) (xy 180.34 139.7)
 		)
@@
 	(wire
 		(pts
+			(xy 207.01 354.33) (xy 298.45 354.33)
+		)
+		(stroke
+			(width 0)
+			(type default)
+		)
+	)
+	(wire
+		(pts
 			(xy 153.67 116.84) (xy 180.34 116.84)
 		)
@@
 	(wire
 		(pts
-			(xy 152.4 359.41) (xy 149.86 359.41)
+			(xy 139.7 365.76) (xy 35.56 365.76)
 		)
 		(stroke
@@
 	(wire
 		(pts
+			(xy 139.7 354.33) (xy 152.4 354.33)
+		)
+		(stroke
+			(width 0)
+			(type default)
+		)
+	)
+	(wire
+		(pts
+			(xy 139.7 365.76) (xy 139.7 359.41)
+		)
+		(stroke
+			(width 0)
+			(type default)
+		)
+	)
+	(wire
+		(pts
 			(xy 161.29 152.4) (xy 161.29 299.72)
 		)
@@
 		)
 	)
-	(polyline
-		(pts
-			(xy 142.24 345.44) (xy 148.59 345.44)
-		)
-		(stroke
-			(width 0)
-			(type default)
-		)
-	)
 	(wire
 		(pts
@@
 		)
 	)
-	(text "It's LOW that's not right?"
-		(exclude_from_sim no)
-		(at 137.414 344.424 0)
-		(effects
-			(font
-				(size 1.27 1.27)
-			)
-		)
-	)
 	(text "Write: MDP is \"1\"\nRead: MDP is the parity bit"
 		(exclude_from_sim no)
@@
 		)
 	)
-	(label "nHRQDMA"
-		(at 212.09 354.33 0)
-		(effects
-			(font
-				(size 1.27 1.27)
-			)
-			(justify left bottom)
-		)
-	)
 	(label "XD7"
 		(at 533.4 419.1 180)
@@
 		)
 	)
-	(label "HOLDA"
-		(at 149.86 359.41 180)
-		(effects
-			(font
-				(size 1.27 1.27)
-			)
-			(justify right bottom)
-		)
-	)
 	(label "XD1"
 		(at 80.01 383.54 180)
@@
 		)
 	)
-	(label "RDYTODMA"
-		(at 149.86 354.33 180)
-		(effects
-			(font
-				(size 1.27 1.27)
-			)
-			(justify right bottom)
-		)
-	)
 	(label "nCMDEN?"
 		(at 267.97 288.29 180)
@@
 		)
 	)
-	(label "DRQ0"
-		(at 152.4 369.57 180)
-		(effects
-			(font
-				(size 1.27 1.27)
-			)
-			(justify right bottom)
-		)
-	)
 	(label "U5917_373_OE"
 		(at 659.13 154.94 0)
@@
 		)
 	)
+	(global_label "DRQ0"
+		(shape input)
+		(at 35.56 369.57 180)
+		(fields_autoplaced yes)
+		(effects
+			(font
+				(size 1.27 1.27)
+			)
+			(justify right)
+		)
+		(property "Intersheetrefs" "${INTERSHEET_REFS}"
+			(at 27.4948 369.57 0)
+			(effects
+				(font
+					(size 1.27 1.27)
+				)
+				(justify right)
+				(hide yes)
+			)
+		)
+	)
 	(global_label "S1"
 		(shape input)
@@
 		)
 	)
+	(global_label "HOLDA"
+		(shape input)
+		(at 35.56 365.76 180)
+		(fields_autoplaced yes)
+		(effects
+			(font
+				(size 1.27 1.27)
+			)
+			(justify right)
+		)
+		(property "Intersheetrefs" "${INTERSHEET_REFS}"
+			(at 26.5271 365.76 0)
+			(effects
+				(font
+					(size 1.27 1.27)
+				)
+				(justify right)
+				(hide yes)
+			)
+		)
+	)
 	(global_label "A0"
 		(shape output)
@@
 		)
 	)
+	(global_label "nHRQDMA"
+		(shape output)
+		(at 298.45 354.33 0)
+		(fields_autoplaced yes)
+		(effects
+			(font
+				(size 1.27 1.27)
+			)
+			(justify left)
+		)
+		(property "Intersheetrefs" "${INTERSHEET_REFS}"
+			(at 310.3252 354.33 0)
+			(effects
+				(font
+					(size 1.27 1.27)
+				)
+				(justify left)
+				(hide yes)
+			)
+		)
+	)
 	(global_label "nXIOW"
 		(shape input)
@@
 			(effects
 				(font
+					(size 1.27 1.27)
+				)
+				(justify right)
+				(hide yes)
+			)
+		)
+	)
+	(global_label "RDYTODMA"
+		(shape input)
+		(at 34.29 344.17 180)
+		(fields_autoplaced yes)
+		(effects
+			(font
+				(size 1.27 1.27)
+			)
+			(justify right)
+		)
+		(property "Intersheetrefs" "${INTERSHEET_REFS}"
+			(at 21.5681 344.17 0)
+			(effects
+				(font

Commit message: Little tidy up
Parts:
- renumbered U28 to U5716, U29 to U5916
Connections:
- net PCLK: now also U9.2 (PCLK)
Changed lines of the file:
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@@
 	(wire
 		(pts
+			(xy 67.31 45.72) (xy 60.96 45.72)
+		)
+		(stroke
+			(width 0)
+			(type default)
+		)
+	)
+	(wire
+		(pts
 			(xy 773.43 468.63) (xy 770.89 468.63)
 		)
@@
 	(wire
 		(pts
-			(xy 144.78 463.55) (xy 156.21 463.55)
+			(xy 144.78 463.55) (xy 185.42 463.55)
 		)
 		(stroke
@@
 	(wire
 		(pts
+			(xy 113.03 431.8) (xy 161.29 431.8)
+		)
+		(stroke
+			(width 0)
+			(type default)
+		)
+	)
+	(wire
+		(pts
 			(xy 604.52 78.74) (xy 660.4 78.74)
 		)
@@
 	(wire
 		(pts
+			(xy 161.29 461.01) (xy 144.78 461.01)
+		)
+		(stroke
+			(width 0)
+			(type default)
+		)
+	)
+	(wire
+		(pts
 			(xy 628.65 82.55) (xy 628.65 83.82)
 		)
@@
 	(wire
 		(pts
+			(xy 161.29 431.8) (xy 161.29 461.01)
+		)
+		(stroke
+			(width 0)
+			(type default)
+		)
+	)
+	(wire
+		(pts
 			(xy 336.55 40.64) (xy 363.22 40.64)
 		)
@@
 	(wire
 		(pts
-			(xy 144.78 461.01) (xy 185.42 461.01)
-		)
-		(stroke
-			(width 0)
-			(type default)
-		)
-	)
-	(wire
-		(pts
 			(xy 492.76 289.56) (xy 455.93 289.56)
 		)
@@
 		)
 	)
+	(label "8253_CLKS"
+		(at 185.42 463.55 0)
+		(effects
+			(font
+				(size 1.27 1.27)
+			)
+			(justify left bottom)
+		)
+	)
 	(label "A18"
 		(at 243.84 360.68 180)
@@
 		)
 	)
-	(label "8253_CLKS"
-		(at 156.21 463.55 0)
-		(effects
-			(font
-				(size 1.27 1.27)
-			)
-			(justify left bottom)
-		)
-	)
 	(label "5716_245_DIR"
 		(at 533.4 471.17 180)
@@
 		)
 	)
-	(global_label "PCLK"
-		(shape output)
-		(at 185.42 461.01 0)
-		(fields_autoplaced yes)
-		(effects
-			(font
-				(size 1.27 1.27)
-			)
-			(justify left)
-		)
-		(property "Intersheetrefs" "${INTERSHEET_REFS}"
-			(at 193.2433 461.01 0)
-			(effects
-				(font
-					(size 1.27 1.27)
-				)
-				(justify left)
-				(hide yes)
-			)
-		)
-	)
 	(global_label "BUF_CLK_INV"
 		(shape input)
@@
 		)
 	)
+	(global_label "PCLK"
+		(shape input)
+		(at 113.03 431.8 180)
+		(fields_autoplaced yes)
+		(effects
+			(font
+				(size 1.27 1.27)
+			)
+			(justify right)
+		)
+		(property "Intersheetrefs" "${INTERSHEET_REFS}"
+			(at 105.2067 431.8 0)
+			(effects
+				(font
+					(size 1.27 1.27)
+				)
+				(justify right)
+				(hide yes)
+			)
+		)
+	)
 	(global_label "nDMAWAIT?"
 		(shape input)
@@
 		)
 	)
+	(global_label "PCLK"
+		(shape output)
+		(at 67.31 45.72 0)
+		(fields_autoplaced yes)
+		(effects
+			(font
+				(size 1.27 1.27)
+			)
+			(justify left)
+		)
+		(property "Intersheetrefs" "${INTERSHEET_REFS}"
+			(at 75.1333 45.72 0)
+			(effects
+				(font
+					(size 1.27 1.27)
+				)
+				(justify left)
+				(hide yes)
+			)
+		)
+	)
 	(global_label "RD_nP_ERROR_LO{slash}WR_MDP_LO"
 		(shape input)
@@
 		(dnp no)
 		(fields_autoplaced yes)
-		(property "Reference" "U28"
+		(property "Reference" "U5716"
 			(at 548.2941 440.69 0)
 			(effects
@@
 			(project "FerrantiPC33"
 				(path "/69e7ee7f-eba6-467b-99f5-85e34f143cc1"
-					(reference "U28")
+					(reference "U5716")
 					(unit 1)
 				)
@@
 		(dnp no)
 		(fields_autoplaced yes)
-		(property "Reference" "U29"
+		(property "Reference" "U5916"
 			(at 548.2941 490.22 0)
 			(effects
@@
 			(project "FerrantiPC33"
 				(path "/69e7ee7f-eba6-467b-99f5-85e34f143cc1"
-					(reference "U29")
+					(reference "U5916")
 					(unit 1)
 				)
@@
 		(on_board yes)
 		(dnp no)
-		(fields_autoplaced yes)
 		(property "Reference" "C1"
-			(at 74.93 48.26 90)
+			(at 77.978 51.816 90)
 			(effects
 				(font
@@
 		)
 		(property "Value" "45pF"
-			(at 74.93 50.8 90)
+			(at 78.994 53.848 90)
 			(effects
 				(font
